File: dimmer-pcb.kicad_pcb (KiCad board)
At the start: 2 copper layers, 13 parts, among them J3 Conn_01x04, Q1 BT136, U1 PC817, U3 MOC3021

Commit message: Add files via upload
Other:
- board text added: "Fan"
Changed lines of the file:
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@@
+		)
+	)
+	(gr_text "Fan"
+		(at 89.31 129.73 0)
+		(layer "F.Fab")
+		(effects
+			(font
+				(size 0.8 0.8)
+				(thickness 0.15)
+			)
+			(justify left bottom)
 		)
 	)
@@
 		(layer "F.Fab")
 		(effects
-			(font
-				(size 1 1)
-				(thickness 0.15)
-			)
-			(justify left bottom)
-		)
-	)
-	(gr_text "L"
-		(at 89.52 130.213 0)
-		(layer "F.Fab")
-		(effects

Commit message: Add files via upload
Other:
- board outline added: 53.2 x 29.7 mm
Changed lines of the file:
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@@
 		(filling no)
 		(pcbplotparams
-			(layerselection 0x00000000_00000000_5555555d_5555557c)
+			(layerselection 0x00000000_00000000_5555555d_5755557c)
 			(plot_on_all_layers_selection 0x00000000_00000000_00000000_00000000)
 			(disableapertmacros no)
@@
 		(layer "F.SilkS")
 	)
+	(gr_rect
+		(start 89.17 106.42)
+		(end 142.33 136.08)
+		(stroke
+			(width 0.05)
+			(type default)
+		)
+		(fill no)
+		(layer "Edge.Cuts")
+	)
 	(gr_text "SASoftwareS"
