File: dimmer-pcb.kicad_pcb (KiCad board)
At the start: 2 copper layers, 53.2 x 29.7 mm, 13 parts, among them J3 Conn_01x04, Q1 BT136, U1 PC817, U3 MOC3021

Commit message: Add files via upload
Parts:
- C1: footprint Capacitor_THT:C_Disc_D16.0mm_W5.0mm_P10.00mm -> Capacitor_THT:C_Rect_L18.0mm_W6.0mm_P15.00mm_FKS3_FKP3
- U3: value MOC3021 -> MOC3021M
- moved Q1 3.51 mm to (100.5, 124.0)
- moved J1 2.61 mm to (92.9, 112.6)
- moved J2 2.61 mm to (92.9, 124.1)
- moved C1 0.45 mm to (122.2, 123.6)
- renumbered DB107 to BR1
Routing:
- net Net-(J1-Pin_1): track 42.8 -> 49.0 mm
- net Net-(J1-Pin_2): track 21.9 -> 24.5 mm
- net Net-(J2-Pin_2): track 27.6 -> 30.3 mm
- net Net-(Q1-G): track 39.7 -> 41.3 mm
Other:
- board size 53.2 x 29.7 mm -> 58.3 x 29.5 mm
Changed lines of the file:
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@@
 	(footprint "TerminalBlock:TerminalBlock_MaiXu_MX126-5.0-02P_1x02_P5.00mm"
 		(layer "F.Cu")
-		(at 95.5 112.5 -90)
+		(at 92.89 112.56 -90)
 		(descr "terminal block MaiXu MX126-5.0-02P, 2 pins, pitch 5mm, size 10.5x7.8mm, drill diameter 1.3mm, pad diameter 2.8mm, https://www.lcsc.com/datasheet/lcsc_datasheet_2309150913_MAX-MX126-5-0-03P-GN01-Cu-S-A_C5188435.pdf")
 		(tags "THT terminal block MaiXu MX126-5.0-02P pitch 5mm size 10.5x7.8mm drill 1.3mm pad 2.8mm")
@@
 	(footprint "Package_TO_SOT_THT:TO-220-3_Vertical"
 		(layer "F.Cu")
-		(at 104.05 123.96 -90)
+		(at 100.54 123.96 -90)
 		(descr "TO-220-3, Vertical, RM 2.54mm, see https://www.vishay.com/docs/66542/to-220-1.pdf")
 		(tags "TO-220-3 Vertical RM 2.54mm")
@@
 			)
 		)
-		(property "Value" "MOC3021"
+		(property "Value" "MOC3021M"
 			(at 3.81 7.41 0)
 			(layer "F.SilkS")
@@
 		)
 	)
-	(footprint "Capacitor_THT:C_Disc_D16.0mm_W5.0mm_P10.00mm"
+	(footprint "Capacitor_THT:C_Rect_L18.0mm_W6.0mm_P15.00mm_FKS3_FKP3"
 		(layer "F.Cu")
-		(at 121.75 123.5 180)
-		(descr "C, Disc series, Radial, pin pitch=10.00mm, diameter*width=16.0*5.0mm^2, Capacitor, http://www.vishay.com/docs/28535/vy2series.pdf")
-		(tags "C Disc series Radial pin pitch 10.00mm diameter 16.0mm width 5.0mm Capacitor")
+		(at 122.19 123.59 180)
+		(descr "C, Rect series, Radial, pin pitch=15.00mm, length*width=18*6mm^2, Capacitor, http://www.wima.com/EN/WIMA_FKS_3.pdf")
+		(tags "C Rect series Radial pin pitch 15.00mm length 18mm width 6mm Capacitor")
 		(property "Reference" "C1"
-			(at 5 -3.75 0)
+			(at 7.5 -4.25 0)
 			(layer "F.SilkS")
-			(hide yes)
 			(effects
 				(font
@@
 		)
 		(property "Value" "104J"
-			(at 5 0 0)
-			(layer "F.SilkS")
+			(at 7.5 4.25 0)
+			(layer "F.Fab")
 			(effects
 				(font
@@
 		(duplicate_pad_numbers_are_jumpers no)
 		(fp_line
-			(start 13.12 2.62)
-			(end -3.12 2.62)
+			(start 16.62 3.12)
+			(end -1.62 3.12)
 			(stroke
 				(width 0.12)
@@
 		)
 		(fp_line
-			(start 13.12 -2.62)
-			(end 13.12 2.62)
+			(start 16.62 -3.12)
+			(end 16.62 3.12)
 			(stroke
 				(width 0.12)
@@
 		)
 		(fp_line
-			(start -3.12 2.62)
-			(end -3.12 -2.62)
+			(start -1.62 3.12)
+			(end -1.62 -3.12)
 			(stroke
 				(width 0.12)
@@
 		)
 		(fp_line
-			(start -3.12 -2.62)
-			(end 13.12 -2.62)
+			(start -1.62 -3.12)
+			(end 16.62 -3.12)
 			(stroke
 				(width 0.12)
@@
 		)
 		(fp_rect
-			(start -3.25 -2.75)
-			(end 13.25 2.75)
+			(start -1.75 -3.25)
+			(end 16.75 3.25)
 			(stroke
 				(width 0.05)
@@
 		)
 		(fp_rect
-			(start -3 -2.5)
-			(end 13 2.5)
+			(start -1.5 -3)
+			(end 16.5 3)
 			(stroke
 				(width 0.1)
@@
 		)
 		(fp_text user "${REFERENCE}"
-			(at 5.23 1.64 0)
+			(at 7.5 0 0)
 			(layer "F.Fab")
 			(effects
@@
 		(pad "1" thru_hole circle
 			(at 0 0 180)
-			(size 2 2)
-			(drill 1)
+			(size 2.4 2.4)
+			(drill 1.2)
 			(layers "*.Cu" "*.Mask")
 			(remove_unused_layers no)
@@
 		)
 		(pad "2" thru_hole circle
-			(at 10 0 180)
-			(size 2 2)
-			(drill 1)
+			(at 15 0 180)
+			(size 2.4 2.4)
+			(drill 1.2)
 			(layers "*.Cu" "*.Mask")
 			(remove_unused_layers no)
@@
 		)
 		(embedded_fonts no)
-		(model "${KICAD10_3DMODEL_DIR}/Capacitor_THT.3dshapes/C_Rect_L13.5mm_W5.0mm_P10.00mm_FKS3_FKP3_MKS4.step"
+		(model "${KICAD10_3DMODEL_DIR}/Capacitor_THT.3dshapes/C_Rect_L18.0mm_W6.0mm_P15.00mm_FKS3_FKP3.step"
 			(offset
 				(xyz 0 0 0)
@@
 	(footprint "TerminalBlock:TerminalBlock_MaiXu_MX126-5.0-02P_1x02_P5.00mm"
 		(layer "F.Cu")
-		(at 95.5 124 -90)
+		(at 92.89 124.06 -90)
 		(descr "terminal block MaiXu MX126-5.0-02P, 2 pins, pitch 5mm, size 10.5x7.8mm, drill diameter 1.3mm, pad diameter 2.8mm, https://www.lcsc.com/datasheet/lcsc_datasheet_2309150913_MAX-MX126-5-0-03P-GN01-Cu-S-A_C5188435.pdf")
 		(tags "THT terminal block MaiXu MX126-5.0-02P pitch 5mm size 10.5x7.8mm drill 1.3mm pad 2.8mm")
@@
 		(layer "F.Cu")
 		(at 115 115 180)
-		(property "Reference" "DB107"
+		(property "Reference" "BR1"
 			(at -0.645 -5.635 0)
 			(layer "F.SilkS")
@@
 		(sheetname "/")
 		(sheetfile "dimmer-pcb.kicad_sch")
+		(units
+			(unit
+				(name "A")
+				(pins "1" "3" "4" "2")
+			)
+		)
 		(attr through_hole)
 		(duplicate_pad_numbers_are_jumpers no)
@@
 	(gr_poly
 		(pts
-			(xy 94.96 124.02) (xy 96.13 124.02) (xy 96.13 117.58) (xy 94.87 117.58) (xy 94.86 124.02) (xy 94.89 124.02)
+			(xy 92.35 124.08) (xy 93.52 124.08) (xy 93.52 117.64) (xy 92.26 117.64) (xy 92.25 124.08) (xy 92.28 124.08)
 		)
 		(stroke
@@
 	)
 	(gr_rect
-		(start 89.25 106.5)
-		(end 142.25 136)
+		(start 84.28 106.535)
+		(end 142.45 135.845)
 		(stroke
 			(width 0.1)
@@
 	)
 	(gr_rect
-		(start 89.17 106.42)
-		(end 142.33 136.08)
+		(start 84.2 106.44)
+		(end 142.53 135.93)
 		(stroke
 			(width 0.05)
@@
 	)
 	(gr_text "Fan"
-		(at 89.31 129.73 0)
+		(at 84.41 129.83 0)
 		(layer "F.SilkS")
 		(effects
@@
 	)
 	(gr_text "N"
-		(at 89.5 124.64 0)
+		(at 84.6 124.74 0)
 		(layer "F.SilkS")
 		(effects
@@
 	)
 	(gr_text "N"
-		(at 89.53 118.3 0)
+		(at 84.63 118.4 0)
 		(layer "F.SilkS")
 		(effects
@@
 	)
 	(gr_text "L"
-		(at 89.54 113.3 0)
+		(at 84.64 113.4 0)
 		(layer "F.SilkS")
 		(effects
@@
 	)
 	(segment
-		(start 114.5 120.75)
-		(end 111.75 123.5)
+		(start 102.5 112)
+		(end 105 109.5)
 		(width 2)
 		(layer "B.Cu")
@@
 	)
 	(segment
-		(start 102.5 112)
-		(end 105 109.5)
+		(start 92.89 112.56)
+		(end 92.95 112.5)
+		(width 2.5)
+		(layer "B.Cu")
+		(net "Net-(J1-Pin_1)")
+	)
+	(segment
+		(start 100.54 123.96)
+		(end 106.82 123.96)
 		(width 2)
 		(layer "B.Cu")
@@
 	)
 	(segment
-		(start 111.29 123.96)
-		(end 111.75 123.5)
+		(start 92.95 112.5)
+		(end 102.5 112.5)
+		(width 2.5)
+		(layer "B.Cu")
+		(net "Net-(J1-Pin_1)")
+	)
+	(segment
+		(start 111.66 123.59)
+		(end 114.5 120.75)
 		(width 2)
 		(layer "B.Cu")
@@
 	)
 	(segment
-		(start 104.05 123.96)
-		(end 111.29 123.96)
+		(start 114.5 110.75)
+		(end 114.5 120.75)
 		(width 2)
 		(layer "B.Cu")
@@
 	)
 	(segment
-		(start 114.5 110.75)
-		(end 114.5 120.75)
+		(start 107.19 123.59)
+		(end 111.66 123.59)
 		(width 2)
 		(layer "B.Cu")
@@
 	)
 	(segment
-		(start 95.5 112.5)
-		(end 102.5 112.5)
-		(width 2.5)
+		(start 106.82 123.96)
+		(end 107.19 123.59)
+		(width 2)
 		(layer "B.Cu")
 		(net "Net-(J1-Pin_1)")
@@
 	)
 	(segment
-		(start 110.825 117.5)
-		(end 110.875 117.55)
+		(start 92.95 117.5)
+		(end 110.825 117.5)
 		(width 2.5)
 		(layer "B.Cu")
@@
 	)
 	(segment
-		(start 95.5 117.5)
-		(end 110.825 117.5)
+		(start 92.89 117.56)
+		(end 92.95 117.5)
 		(width 2.5)
 		(layer "B.Cu")
@@
 	)
 	(segment
-		(start 95.5 117.5)
-		(end 95.5 124)
+		(start 110.825 117.5)
+		(end 110.875 117.55)
+		(width 2.5)
+		(layer "B.Cu")
+		(net "Net-(J1-Pin_2)")
+	)
+	(segment
+		(start 92.89 117.56)
+		(end 92.89 124.06)
 		(width 2.5)
 		(layer "B.Cu")
@@
 	)
 	(segment
-		(start 98.44 129)
-		(end 100.94 126.5)
+		(start 98.39 126.5)
+		(end 95.83 129.06)
 		(width 2)
 		(layer "B.Cu")
@@
 	)
 	(segment
-		(start 95.5 129)
-		(end 98.44 129)
+		(start 92.89 129.06)
+		(end 95.83 129.06)
 		(width 2)
 		(layer "B.Cu")
@@
 	)
 	(segment
-		(start 104.05 126.5)
+		(start 100.54 126.5)
 		(end 107.75 126.5)
 		(width 2)
@@
 	)
 	(segment
-		(start 100.94 126.5)
-		(end 104.05 126.5)
-		(width 2)
-		(layer "B.Cu")
-		(net "Net-(J2-Pin_2)")
-	)
-	(segment
 		(start 119.205 129)
 		(end 117.005 131.2)
@@
 	)
 	(segment
-		(start 107.75 126.5)
-		(end 110.5 129.25)
+		(start 100.54 126.5)
+		(end 98.39 126.5)
 		(width 2)
 		(layer "B.Cu")
@@
 	)
 	(segment
-		(start 127.19 125.46)
-		(end 129.46 125.46)
+		(start 107.75 126.5)
+		(end 110.5 129.25)
 		(width 2)
 		(layer "B.Cu")
-		(net "Net-(Q1-G)")
+		(net "Net-(J2-Pin_2)")
 	)
 	(segment
-		(start 131 127)
-		(end 131 130.5)
+		(start 129.46 125.46)
+		(end 131 127)
 		(width 2)
 		(layer "B.Cu")
@@
 	(segment
 		(start 128.25 133.25)
-		(end 105 133.25)
+		(end 108.04 133.25)
 		(width 2)
 		(layer "B.Cu")
@@
 	)
 	(segment
-		(start 129.46 125.46)
-		(end 131 127)
+		(start 127.19 125.46)
+		(end 129.46 125.46)
 		(width 2)
 		(layer "B.Cu")
@@
 	)
 	(segment
-		(start 104.05 132.3)
-		(end 104.05 129.04)
+		(start 103.83 129.04)
+		(end 108.04 133.25)
+		(width 2)
+		(layer "B.Cu")
+		(net "Net-(Q1-G)")
+	)
+	(segment
+		(start 100.54 129.04)
+		(end 103.83 129.04)
 		(width 2)
 		(layer "B.Cu")
@@
 	)
 	(segment
-		(start 105 133.25)
-		(end 104.05 132.3)
+		(start 131 127)
+		(end 131 130.5)
 		(width 2)
 		(layer "B.Cu")
@@
 	)
 	(segment
-		(start 121.75 123.5)
-		(end 118 123.5)
+		(start 122.19 123.59)
+		(end 117.91 123.59)
 		(width 2)
 		(layer "B.Cu")
@@
 	)
 	(segment
-		(start 118 123.5)
+		(start 117.91 123.59)
 		(end 115.58 125.92)
 		(width 2)
