File: dimmer-pcb.kicad_sch (KiCad schematic)
At the start: 13 parts, among them J3 Conn_01x04, Q1 BT136, U1 PC817, U3 MOC3021M

Commit message: Add files via upload
Parts:
- C1: footprint Capacitor_THT:C_Disc_D16.0mm_W5.0mm_P10.00mm -> Capacitor_THT:C_Rect_L18.0mm_W6.0mm_P15.00mm_FKS3_FKP3
Changed lines of the file:
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@@
 			)
 		)
-		(property "Footprint" "Capacitor_THT:C_Disc_D16.0mm_W5.0mm_P10.00mm"
+		(property "Footprint" "Capacitor_THT:C_Rect_L18.0mm_W6.0mm_P15.00mm_FKS3_FKP3"
 			(at 164.7952 111.76 0)
 			(hide yes)
